File: pcb/scales_stepper_stm32/scales_stepper_stm32.kicad_sch (KiCad schematic)
At the start: 25 parts, among them J1 USB_B_Micro, J2 Conn_01x04_Pin, J3 Screw_Terminal_01x02, J4 Screw_Terminal_01x04, SW1 BUTT_JOGL, SW2 BUTT_JOGL, SW3 BUTT_JOGL, SW4 BUTT_JOGL, SW5 BUTT_JOGL, SW6 BUTT_JOGL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

Commit message: morse code
Parts:
- added C5, C6: 100n, Capacitor_SMD:C_0805_2012Metric_Pad1.18x1.45mm_HandSolder, symbol Device:C
- added J5: Screw_Terminal_01x04, TerminalBlock_CUI:TerminalBlock_CUI_TB007-508-04_1x04_P5.08mm_Horizontal, symbol Connector:Screw_Terminal_01x04
Connections:
- net +3V3: now also C5.1, C6.1
- net ES_L: now also J5.1 (Pin_1)
- net ES_R: now also J5.3 (Pin_3)
- net GND: now also C5.2, C6.2, J5.2 (Pin_2), J5.4 (Pin_4)
